File: Version 1/schematic.sch (EAGLE design)
At the start: 52 parts, among them IC1 FT230XS, IC4 L4931D, X1 MINI-USB-32005-301

Commit message: Saving to git
Changed lines of the file:
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@@
 <part name="LED4" library="adafruit" deviceset="LED" device="SMT1206"/>
 <part name="SUPPLY19" library="supply2" deviceset="GND" device=""/>
+<part name="P+5" library="supply1" deviceset="VCC" device=""/>
 </parts>
 <sheets>
@@
 <instance part="LED4" gate="G$1" x="-162.56" y="30.48" rot="R180"/>
 <instance part="SUPPLY19" gate="GND" x="-162.56" y="25.4"/>
+<instance part="P+5" gate="VCC" x="55.88" y="134.62"/>
 </instances>
 <busses>
@@
 <pinref part="C7" gate="G$1" pin="1"/>
 <pinref part="L1" gate="G$1" pin="2"/>
-<wire x1="50.8" y1="132.08" x2="58.42" y2="132.08" width="0.1524" layer="91"/>
+<wire x1="50.8" y1="132.08" x2="55.88" y2="132.08" width="0.1524" layer="91"/>
 <label x="53.34" y="127" size="1.778" layer="95"/>
+<pinref part="P+5" gate="VCC" pin="VCC"/>
+<wire x1="55.88" y1="132.08" x2="58.42" y2="132.08" width="0.1524" layer="91"/>
+<junction x="55.88" y="132.08"/>
 </segment>
 <segment>
@@
 <pinref part="IC1" gate="G$1" pin="3V3OUT"/>
 <wire x1="53.34" y1="121.92" x2="50.8" y2="121.92" width="0.1524" layer="91"/>
+<label x="48.26" y="124.46" size="1.778" layer="95"/>
 </segment>
 <segment>
@@
 <wire x1="48.26" y1="104.14" x2="53.34" y2="104.14" width="0.1524" layer="91"/>
 <junction x="53.34" y="104.14"/>
-</segment>
-<segment>
+<label x="45.72" y="106.68" size="1.778" layer="95"/>
+</segment>
+<segment>
