File: Version 2 PCB Files/2.1/2.1.brd (EAGLE design)
At the start: 37.9 x 37.6 mm, 54 parts, among them IC1 FT230XS, IC4 L4931D, X1 MINI-USB-32005-301

Commit message: saving to git
Parts:
- removed C11: .1uf, rcl:C0603K
- removed C12, C13, C17, C18: 1uF, rcl:C0603K
- removed C14, C15: 2.2uF, rcl:C0603K
- removed C16: .1uF, rcl:C0603K
- removed JP1: (no value), adafruit:1X06-BIG
- removed JP4, JP5: (no value), adafruit:1X01
- removed LED1, LED2, LED3: (no value), adafruit:1206
- removed R12: 2K, eagle-ltspice:R0603
- removed R14: 390K, eagle-ltspice:R0603
- removed R17, R18, R19: 330, eagle-ltspice:R0603
- removed U$4: ATMEGA32U4-AU, adafruit:TQFP44
- added IC2: ATMEGA644A, atmel:TQFP44
- added J1: XF2L-1025-1A, 10pinzif:CON10_1X10_DBR_XF2L
- added JP2: (no value), adafruit:1X06-BIG
- added JP6, JP7: (no value), adafruit:1X01
- added LED5, LED6, LED7: (no value), adafruit:1206
- added R10, R11, R15: 330, eagle-ltspice:R0603
- R13: value 2K -> 100
- U$3: value UG-2864HSWEG01 -> AT45DB641E; device adafruit:1X30-0.7MM -> MyParts:SO08
- moved C19 67.8 mm to (5.73, 27.6), flipped to the bottom, turned to 270 degrees
- moved U$3 62.4 mm to (-37.0, 3.97), flipped to the top, turned to 0 degrees
- moved R5 50.4 mm to (4.13, 27.6), flipped to the bottom, turned to 90 degrees
- moved U$2 47.9 mm to (9.50, 29.7), flipped to the bottom, turned to 90 degrees
- moved D1 40.2 mm to (7.10, 28.5), flipped to the bottom, turned to 90 degrees
- moved C7 34.2 mm to (11.6, 1.86)
- moved C4 33.5 mm to (7.55, 35.4)
- moved R2 24.4 mm to (68.0, 22.0)
- moved R3 24.4 mm to (68.1, 12.4)
- moved R4 24.4 mm to (67.9, 31.6)
- moved LED4 21.1 mm to (13.4, 35.3), turned to 180 degrees
- moved C9 20.4 mm to (12.9, 1.85), flipped to the top, turned to 270 degrees
- moved C8 18.0 mm to (14.2, 1.86), flipped to the top, turned to 270 degrees
- moved C10 18.0 mm to (19.7, 1.39), turned to 180 degrees
- moved C2 16.9 mm to (6.57, 33.9), flipped to the bottom, turned to 180 degrees
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Connections:
- removed net N$10: C13.1, U$3.3
- removed net N$14: C18.2, U$4.6
- removed net N$17: LED1.A, R17.1
- removed net N$18: LED2.A, R18.1
- removed net N$19: LED3.A, R19.1
- removed net N$21: R19.2, U$4.29
- removed net N$22: R18.2, U$4.30
- removed net N$7: C13.2, U$3.2
- removed net N$8: C17.1, U$3.4
- removed net N$9: R14.1, U$3.26
- removed net OLED_SCL: R12.1, U$3.18, U$4.18
- removed net OLED_SDA: R13.1, U$3.19, U$3.20, U$4.19
- new net ANODE: IC2.16, J1.1
- new net CS: IC2.22
- new net KATHODE: J1.2, R13.1
- new net N$11: LED5.A, R10.1
- new net N$12: LED6.A, R11.1
- new net N$13: LED7.A, R15.1
- new net N$15: IC2.13, R15.2
- new net N$16: IC2.14, R11.2
- new net N$20: IC2.15, R10.2
- new net N$24: IC2.10, JP6.1
- new net N$26: J1.12
- new net N$27: J1.11
- new net N1: J1.7
- new net RST: IC2.21
- new net RXD1: IC2.9, JP7.1
- new net SCL: J1.9
- new net SDA: J1.8
- net B0: now also IC2.11; no longer U$4.25
- net B1: now also IC2.12; no longer U$4.22
- net B2: now also IC2.42; no longer U$4.26
- net GND: now also IC2.18, IC2.28, IC2.39, IC2.6, J1.3, J1.5, JP2.6, LED5.C, LED6.C, LED7.C, R13.2; no longer C11.1, C12.1, C14.1, C15.1, C16.1, C18.1, JP1.6, LED1.C, LED2.C, LED3.C, R14.2, U$3.1, U$3.10, U$3.12, U$3.13, U$3.15, U$3.16, U$3.17, U$3.29, U$3.30, U$3.8, U$4.15, U$4.23, U$4.35, U$4.43, U$4.5
- net MISO: now also IC2.2, JP2.3; no longer JP1.3, U$4.11
- net MOSI: now also IC2.1, JP2.4; no longer JP1.4, U$4.10
- net N$23: now also J1.6; no longer R17.2, U$4.12
- net N$5: now also IC2.19; no longer C14.2, U$3.27
- net N$6: now also IC2.20; no longer C17.2, U$3.5
- net RESET: now also IC2.4, JP2.2; no longer JP1.2, U$4.13
- net RXD: no longer JP5.1, U$4.20
- net SCK: now also IC2.3, JP2.5; no longer JP1.5, U$4.9
- net TXD: no longer JP4.1, U$4.21
- net VCC: now also IC2.17, IC2.27, IC2.38, IC2.5, J1.10, J1.4; no longer C11.2, C12.2, C15.2, C16.2, JP1.1, R12.2, R13.2, U$3.11, U$3.14, U$3.28, U$3.6, U$3.9, U$4.14, U$4.24, U$4.34, U$4.44
- net VDD: now also JP2.1
- net VUSB: no longer U$4.2, U$4.7
Routing:
- net GND: track 0.00 -> 50.1 mm, vias 0 -> 5
- net VCC: track 0.00 -> 19.1 mm, vias 0 -> 1
- net NET1: track 0.00 -> 15.8 mm, vias 0 -> 1
- net VDD: track 0.00 -> 12.5 mm
- net 8: track 0.00 -> 10.1 mm, vias 0 -> 1
- net RXD: track 0.00 -> 9.10 mm, vias 0 -> 1
- net VUSB: track 0.00 -> 7.83 mm
- net VBAT: track 0.00 -> 6.42 mm
- net TXD: track 0.00 -> 5.64 mm, vias 0 -> 1
- net USB+: track 0.00 -> 5.48 mm, vias 0 -> 1
- net USB-: track 0.00 -> 5.44 mm
- net 9: track 0.00 -> 4.57 mm
- net N$2: track 0.00 -> 3.62 mm
- net FTDI_VCC: track 0.00 -> 1.73 mm
- net N$1: track 0.00 -> 1.71 mm
Other:
- board size 37.9 x 37.6 mm -> 25.2 x 37.6 mm

Commit message: Added a way to bypass LIPO charging circuitry which wont be ready for the next prototype
Parts:
- JP3: device adafruit:1X03 -> con-lstb:MA04-1
Connections:
- net VDD: now also JP3.4
Changed lines of the file:
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@@
 <attribute name="SPICEPREFIX" value="R" x="22.7507" y="6.3277" size="1.778" layer="28" rot="MR270" display="off"/>
 </element>
-<element name="JP3" library="adafruit" package="1X03" value="" x="1.27" y="15.875" rot="R90"/>
+<element name="JP3" library="con-lstb" package="MA04-1" value="" x="1.27" y="15.875" rot="R90">
+<attribute name="MF" value="" x="1.27" y="15.875" size="1.778" layer="27" rot="R90" display="off"/>
+<attribute name="MPN" value="" x="1.27" y="15.875" size="1.778" layer="27" rot="R90" display="off"/>
+<attribute name="OC_FARNELL" value="unknown" x="1.27" y="15.875" size="1.778" layer="27" rot="R90" display="off"/>
+<attribute name="OC_NEWARK" value="unknown" x="1.27" y="15.875" size="1.778" layer="27" rot="R90" display="off"/>
+</element>
 <element name="LED4" library="adafruit" package="1206" value="" x="13.3658" y="35.3401" rot="R180"/>
 <element name="D1" library="diode" package="SOD323_ST" value="BAT60J" x="7.1" y="28.5171" rot="MR90"/>
@@
 <wire x1="7.446" y1="33.9453" x2="14.7878" y2="35.3401" width="0" layer="19" extent="1-16"/>
 <wire x1="2.75" y1="27.7" x2="2.3875" y2="31.5583" width="0" layer="19" extent="1-1"/>
-<wire x1="1.27" y1="18.415" x2="3.6896" y2="26.7604" width="0" layer="19" extent="16-16"/>
+<wire x1="1.27" y1="17.145" x2="3.6896" y2="26.7604" width="0" layer="19" extent="16-16"/>
 <wire x1="5.4597" y1="48.0936" x2="6.6792" y2="35.4198" width="0" layer="19" extent="1-1"/>
 <wire x1="5.4597" y1="55.0936" x2="5.4597" y2="48.0936" width="0" layer="19" extent="1-1"/>
 <wire x1="11.4597" y1="55.0936" x2="5.4597" y2="55.0936" width="0" layer="19" extent="1-1"/>
-<wire x1="8.715" y1="5.55" x2="1.27" y2="18.415" width="0" layer="19" extent="1-1"/>
+<wire x1="8.715" y1="5.55" x2="1.27" y2="17.145" width="0" layer="19" extent="1-1"/>
 <wire x1="34.8837" y1="2.8481" x2="22.505" y2="5.1525" width="0" layer="19" extent="1-16"/>
 <wire x1="35.8837" y1="2.8481" x2="34.8837" y2="2.8481" width="0" layer="19" extent="16-16"/>
@@
 <wire x1="5.4796" y1="30.3581125" x2="5.4796" y2="29.8178" width="0.1524" layer="16"/>
 <wire x1="4.0318" y1="31.8059125" x2="5.4796" y2="30.3581125" width="0.1524" layer="16"/>
-<wire x1="1.27" y1="13.335" x2="5.4796" y2="29.8178" width="0" layer="19" extent="16-16"/>
-<wire x1="8.715" y1="7.95" x2="1.27" y2="13.335" width="0" layer="19" extent="1-1"/>
+<wire x1="1.27" y1="12.065" x2="5.4796" y2="29.8178" width="0" layer="19" extent="16-16"/>
+<wire x1="8.715" y1="7.95" x2="1.27" y2="12.065" width="0" layer="19" extent="1-1"/>
 </signal>
 <signal name="FTDI_VCC">
@@
 <wire x1="6.4715125" y1="31.8729" x2="5.7834125" y2="32.561" width="0.1524" layer="16"/>
 <wire x1="5.4796" y1="32.561" x2="5.696" y2="33.9453" width="0" layer="19" extent="16-16"/>
-<wire x1="1.27" y1="15.875" x2="10.7001" y2="29.6691" width="0" layer="19" extent="16-16"/>
+<wire x1="1.27" y1="14.605" x2="10.7001" y2="29.6691" width="0" layer="19" extent="16-16"/>
 </signal>
 <signal name="VDD">
@@
 <wire x1="7.6337" y1="29.0924875" x2="6.9178875" y2="29.8083" width="0.1524" layer="1"/>
 <wire x1="6.9178875" y1="29.8083" x2="2.3875" y2="29.8083" width="0.1524" layer="1"/>
+<contactref element="JP3" pad="4"/>
 <wire x1="8.3001" y1="28.7191" x2="64.65" y2="94" width="0" layer="19" extent="16-16"/>
 <wire x1="7.6337" y1="28.6392" x2="8.3001" y2="28.7191" width="0" layer="19" extent="1-16"/>
+<wire x1="1.27" y1="19.685" x2="4.1305" y2="28.4604" width="0" layer="19" extent="16-16"/>
 </signal>
 <signal name="N$4">

Commit message: Need to layout board and send to fab
Switched to the atmega 328 for simplicity and size, well see what happens, should add an rtc to the board, or a spi header to test the i2c with
Parts:
- removed U$10, U$12, U$13: PUSHBTN, Supply:PUSHBTN
- added U$11, U$4: TL3315NF100Q, MyParts:TL3315NF100Q-PACKAGE
- added U1: ATMEGA328P-AUR32A-L, MyParts:32A-L
- J1: device 10pinzif:CON10_1X10_DBR_XF2L -> MyParts:CON10_1X10_DBR_XF2L
- R13: value 100 -> 160
- U$3: value AT45DB641E -> TL3315NF100Q; device MyParts:SO08 -> MyParts:TL3315NF100Q-PACKAGE
- moved R4 118.6 mm to (-30.6, -34.7), turned to 0 degrees
- moved R3 107.3 mm to (-30.6, -29.9), turned to 0 degrees
- moved U$3 14.2 mm to (-26.9, -6.00)
Connections:
- removed net CS: IC2.22
- removed net N$5: IC2.19
- removed net N$6: IC2.20
- removed net RST: IC2.21
- new net AVCC: U1.18
- new net GND_2: U1.3
- new net GND_3: U1.5
- new net VCC_2: U1.4
- net B0: now also U$3.3, U$3.4; no longer U$12.3, U$12.4
- net B1: now also U$4.3, U$4.4; no longer U$10.3, U$10.4
- net B2: now also U$11.3, U$11.4; no longer U$13.3, U$13.4
- net GND: now also U1.21
- net VCC: now also U$11.1, U$11.2, U$3.1, U$3.2, U$4.1, U$4.2, U1.6; no longer U$10.1, U$10.2, U$12.1, U$12.2, U$13.1, U$13.2

Commit message: Version 2.2 Is finished!
Sent the board to the fab waiting for it.
Parts:
- moved LED4 5.10 mm to (18.5, 35.2)
- moved JP3 2.41 mm to (1.52, 18.3)
