File: Version 2 PCB Files/2.2/2.2.brd (EAGLE design)
At the start: 25.2 x 37.6 mm, 46 parts, among them IC1 FT230XS, IC4 L4931D, J1 XF2L-1025-1A, U1 ATMEGA328P-AUR32A-L, X1 MINI-USB-32005-301

Commit message: Version 2.2 Is finished!
Sent the board to the fab waiting for it.
Parts:
- removed C10, C9: 100nF, rcl:C0603K
- removed C19: 1uF, rcl:C0603K
- removed C5, C6: 47pF, rcl:C0603K
- removed C7: 10nF, rcl:C0603K
- removed C8: 4.7uF, rcl:C0603K
- removed D1: BAT60J, diode:SOD323_ST
- removed IC1: FT230XS, ft230x_10:SSOP16
- removed J1: XF2L-1025-1A, MyParts:CON10_1X10_DBR_XF2L
- removed JP6, JP7: (no value), adafruit:1X01
- removed L1: (no value), inductors:0402
- removed LED5: (no value), adafruit:1206
- removed R10: 330, eagle-ltspice:R0603
- removed R6, R7: 27, eagle-ltspice:R0603
- removed R8, R9: 10K, eagle-ltspice:R0603
- removed U$11, U$3, U$4: TL3315NF100Q, MyParts:TL3315NF100Q-PACKAGE
- removed U$2: 2JS305, SOT346-R:SOT346-R
- removed X1: MINI-USB-32005-301, con-cypressindustries:32005-301
- added C11, C12, C13: 1uF, rcl:C0603K
- added C14: 10nF, rcl:C0603K
- added C15: 4.7uF, rcl:C0603K
- added C16, C17: 100nF, rcl:C0603K
- added D2: BAT60J, diode:SOD323_ST
- added IC2: FT230XS, ft230x_10:SSOP16
- added JP1, JP4: (no value), adafruit:1X03-CLEANBIG
- added L2: (no value), inductors:0402
- added R16: 2K, eagle-ltspice:R0603
- added R17, R20, R21: 10K, eagle-ltspice:R0603
- added R18, R19: 27, eagle-ltspice:R0603
- added U$12: (no value), Microchip_By_element14_Batch_1:SOT95P270X145-5N
- added U$13: 2JS305, SOT346-R:SOT346-R
- added U$5: XF2L-1025-1ABOTTOM, MyParts:CON10_1X10_DBR_XF2L
- added X2: MINI-USB-32005-301, con-cypressindustries:32005-301
- C1, C2: value 1uF -> 47pF
- JP3: device con-lstb:MA04-1 -> adafruit:1X03-CLEANBIG
- R1: value 2K -> 4.7K
- R5: value 10K -> 4.7K
- U$1: value (none) -> M41T62LC6F; device Microchip_By_element14_Batch_1:SOT95P270X145-5N -> MyParts:LCC-8
- moved C1 102.7 mm to (12.9, 5.21), turned to 90 degrees
- moved C2 101.1 mm to (13.3, 5.20), flipped to the bottom, turned to 270 degrees
- moved LED7 97.7 mm to (2.09, 30.2), flipped to the bottom, turned to 270 degrees
- moved R13 88.7 mm to (12.1, 15.7), flipped to the bottom, turned to 90 degrees
- moved R15 80.3 mm to (2.29, 30.2), turned to 270 degrees
- moved R1 79.5 mm to (22.6, 25.8), flipped to the bottom, turned to 90 degrees
- moved R12 79.4 mm to (19.3, 25.6), flipped to the bottom, turned to 90 degrees
- moved R2 77.7 mm to (21.9, 17.3)
- moved JP2 77.1 mm to (2.10, 19.9), turned to 90 degrees
- moved LED6 76.9 mm to (6.39, 24.4), flipped to the bottom
- moved R3 74.2 mm to (21.9, 19.1)
- moved C3 72.5 mm to (14.3, 34.4)
- moved R4 71.2 mm to (21.9, 20.6)
- moved LED4 68.9 mm to (21.9, 31.9), turned to 90 degrees
- moved U1 68.2 mm to (15.5, 21.5), turned to 270 degrees
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Connections:
- removed net FTDI_VCC: IC1.12, L1.1
- removed net KATHODE: J1.2, R13.1
- removed net N$11: LED5.A, R10.1
- removed net N$20: R10.2, U1.11
- new net INT_RTC: U$1.6, U1.1
- new net N$5: R16.2, U$12.5
- new net N$6: R16.1, U$12.2
- new net SCL: R5.1, U$1.8, U1.28
- new net SDA: R1.1, U$1.1, U1.27
- net 8: now also IC2.8, R19.1; no longer IC1.8, R7.1
- net 9: now also IC2.9, R18.1; no longer IC1.9, R6.1
- net B0: now also JP1.1; no longer U$3.3, U$3.4
- net B1: now also JP1.2; no longer U$4.3, U$4.4
- net B2: now also JP1.3; no longer U$11.3, U$11.4
- net GND: now also C1.1, C11.2, C12.2, C13.2, C14.2, C15.2, C16.2, C17.2, IC2.13, IC2.5, JP4.2, R17.1, U$1.3, U$5.6, U$5.8, X2.4; no longer C1.2, C10.2, C19.2, C5.1, C6.2, C7.2, C8.2, C9.2, IC1.13, IC1.5, J1.3, J1.5, LED5.C, R5.1, X1.4
- net LCD_RESET: now also U$5.4; no longer J1.7
- net LEDANODE: now also U$5.10; no longer J1.1
- net MOSI: now also U$5.3; no longer J1.8
- net N$1: now also R13.1, U$5.9; no longer R1.2, U$1.5
- net N$2: now also IC2.12, L2.1; no longer R1.1, U$1.2
- net N$26: now also U$5.12; no longer J1.12
- net N$27: now also U$5.11; no longer J1.11
- net NET1: now also C17.1, IC2.10, IC2.11, IC2.3, R20.1, R21.1; no longer C10.1, IC1.10, IC1.11, IC1.3, R8.1, R9.1
- net RXD: now also IC2.1, R20.2; no longer IC1.1, JP7.1, R8.2
- net SCK: now also U$5.2; no longer J1.9
- net SHEILD: now also X2.5; no longer X1.5
- net SS: now also U$5.5; no longer J1.6
- net TXD: now also IC2.4, R21.2; no longer IC1.4, JP6.1, R9.2
- net USB+: now also C2.1, R19.2, X2.3; no longer C6.1, R7.2, X1.3
- net USB-: now also C1.2, R18.2, X2.2; no longer C5.2, R6.2, X1.2
- net VBAT: now also C12.1, U$12.3, U$13.3; no longer C2.1, U$1.3, U$2.3
- net VCC: now also C14.1, C15.1, C16.1, JP4.1, L2.2, R1.2, R5.2, U$1.5, U$5.1, U$5.7; no longer C7.1, C8.1, C9.1, J1.10, J1.4, L1.2, U$11.1, U$11.2, U$3.1, U$3.2, U$4.1, U$4.2
- net VDD: now also C13.1, D2.C, R17.2, U$13.1; no longer C19.1, D1.C, JP3.4, R5.2, U$2.1
- net VUSB: now also C11.1, D2.A, U$12.1, U$12.4, U$13.2, X2.1; no longer C1.1, D1.A, U$1.1, U$1.4, U$2.2, X1.1
Routing:
- net N$4: track 218.8 -> 0.00 mm
- net GND: track 0.00 -> 134.6 mm, vias 0 -> 12
- net VCC: track 0.00 -> 84.9 mm, vias 0 -> 4
- net VUSB: track 0.00 -> 77.4 mm, vias 0 -> 5
- net VDD: track 0.00 -> 38.4 mm, vias 0 -> 3
- net RXD: track 0.00 -> 32.0 mm, vias 0 -> 3
- net TXD: track 0.00 -> 28.6 mm, vias 0 -> 3
- net VBAT: track 0.00 -> 26.8 mm, vias 0 -> 1
- net SCK: track 0.00 -> 22.4 mm, vias 0 -> 1
- net MOSI: track 0.00 -> 21.4 mm, vias 0 -> 1
- net RESET: track 0.00 -> 19.1 mm, vias 0 -> 2
- net LCD_RESET: track 0.00 -> 17.2 mm, vias 0 -> 1
- net NET1: track 0.00 -> 15.8 mm, vias 0 -> 1
- net SS: track 0.00 -> 15.7 mm, vias 0 -> 1
- net N$3: track 0.00 -> 15.0 mm, vias 0 -> 2
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Other:
- board size 25.2 x 37.6 mm -> 25.9 x 37.9 mm
- board text added: "B0"
- board text added: "B1"
- board text added: "B2"
- board text added: "GND"
- board text added: "MISO"
- board text added: "MOSI"
- board text added: "RESET"
- board text added: "SCK"
- board text added: "VBAT"
- board text added: "VCC"
- board text added: "VDD"
- board text added: "VUSB"
