File: Version 2 PCB Files/2.2/2.2.sch (EAGLE design)
At the start: 45 parts, among them IC1 FT230XS, IC2 ATMEGA644A, IC4 L4931D, J1 XF2L-1025-1A, U1 ATMEGA328P-AUR32A-L, X1 MINI-USB-32005-301

Commit message: Need to layout board and send to fab
Switched to the atmega 328 for simplicity and size, well see what happens, should add an rtc to the board, or a spi header to test the i2c with
Parts:
- removed IC2: ATMEGA644A, atmel:ATMEGA644A
- added R12, R14: 10K, eagle-ltspice:RR0603
- R13: value 160 -> 100
Connections:
- removed net ANODE: IC2.(PCINT31/OC2A)PD7, J1.1(LEDANODE)
- removed net N$15: IC2.(PCINT28/OC1B)PD4, R15.2
- removed net N$23: J1.6(CS)
- removed net N$24: IC2.(PCINT25/TXD0)PD1, JP6.1
- removed net N1: J1.7(RST)
- removed net RXD1: IC2.(PCINT24/RXD0)PD0, JP7.1
- removed net SCL: J1.9(SCL)
- removed net SDA: J1.8(SDA)
- new net LCD_RESET: J1.7(RST), U1.(PCINT1/OC1A)_PB1
- new net LEDANODE: J1.1(LEDANODE), U1.(PCINT0/CLKO/ICP1)_PB0
- new net N$17: U1.AVCC
- new net N$3: R15.2, U1.(PCINT21/OC0B/T1)_PD5
- new net SS: J1.6(CS), R14.2, U1.(PCINT2/SS/OC1B)_PB2
- net B0: now also U1.PC0_(ADC0/PCINT8); no longer IC2.(PCINT26/INT0)PD2
- net B1: now also U1.PC1_(ADC1/PCINT9); no longer IC2.(PCINT27/INT1)PD3
- net B2: now also U1.PC2_(ADC2/PCINT10); no longer IC2.(PCINT10/INT2/AIN0)PB2
- net GND: now also R12.2, U1.GND, U1.GND_2, U1.GND_3; no longer IC2.GND, IC2.GND@1, IC2.GND@2, IC2.GND@3
- net MISO: now also U1.(PCINT4/MISO)_PB4; no longer IC2.(PCINT14/MISO)PB6
- net MOSI: now also J1.8(SDA), U1.(PCINT3/OC2A/MOSI)_PB3; no longer IC2.(PCINT13/MOSI)PB5
- net N$16: now also U1.(PCINT22/OC0A/AIN0)_PD6; no longer IC2.(PCINT29/OC1A)PD5
- net N$20: now also U1.(PCINT23/AIN1)_PD7; no longer IC2.(PCINT30/OC2B/ICP)PD6
- net RESET: now also U1.PC6_(RESET/PCINT14); no longer IC2.RESET
- net RXD: now also JP7.1, U1.PD0_(RXD/PCINT16)
- net SCK: now also J1.9(SCL), U1.PB5_(SCK/PCINT5); no longer IC2.(PCINT15/SCK)PB7
- net TXD: now also JP6.1, U1.PD1_(TXD/PCINT17)
- net VCC: now also R14.1, U1.VCC, U1.VCC_2; no longer IC2.AVCC, IC2.VCC, IC2.VCC@1, IC2.VCC@2
- net VUSB: now also R12.1, U1.PD2_(INT0/PCINT18)
Other:
- note added: "Extra Serial Connection"
- note added: "ISP Header"
- note added: "LCD Display"
- note added: "Microcontroller (ATMEGA 328)"
- note added: "USB Connection"
- moved on the sheet: J1, JP2, JP3, JP6, JP7, LED4, LED5, LED6, LED7, R10, R11, R13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

Commit message: Version 2.2 Is finished!
Sent the board to the fab waiting for it.
Parts:
- removed C10, C9: 100nF, rcl:C-EUC0603K
- removed C5, C6: 47pF, rcl:C-EUC0603K
- removed C7: 10nF, rcl:C-EUC0603K
- removed C8: 4.7uF, rcl:C-EUC0603K
- removed IC1: FT230XS, ft230x_10:FT230XS
- removed J1: XF2L-1025-1A, MyParts:XF2L-1025-1A
- removed JP6, JP7: (no value), adafruit:PINHD-1X1
- removed L1: BLM15HB221SN1, inductors:BLM15HB221SN1
- removed LED5: (no value), adafruit:LEDSMT1206
- removed R10: 330, eagle-ltspice:RR0603
- removed R6, R7: 27, eagle-ltspice:RR0603
- removed R8, R9: 10K, eagle-ltspice:RR0603
- removed U$11, U$3, U$4: TL3315NF100Q, MyParts:TL3315NF100Q
- removed X1: MINI-USB-32005-301, con-cypressindustries:MINI-USB-32005-301
- added C11, C12: 1uF, rcl:C-EUC0603K
- added C14: 10nF, rcl:C-EUC0603K
- added C15: 4.7uF, rcl:C-EUC0603K
- added C16, C17: 100nF, rcl:C-EUC0603K
- added IC2: FT230XS, ft230x_10:FT230XS
- added JP1, JP4: (no value), adafruit:PINHD-1X3CB
- added L2: BLM15HB221SN1, inductors:BLM15HB221SN1
- added R16: 2K, eagle-ltspice:RR0603
- added R17, R20, R21: 10K, eagle-ltspice:RR0603
- added R18, R19: 27, eagle-ltspice:RR0603
- added U$12: MCP73812T-420I/OT, Microchip_By_element14_Batch_1:MCP73812T-420I/OT
- added U$5: XF2L-1025-1ABOTTOM, MyParts:XF2L-1025-1ABOTTOM
- added X2: MINI-USB-32005-301, con-cypressindustries:MINI-USB-32005-301
- C1, C2: value 1uF -> 47pF
- JP3: device con-lstb:MA04-1 -> adafruit:PINHD-1X3CB
- R1: value 2K -> 4.7K
- R5: value 10K -> 4.7K
- U$1: value MCP73812T-420I/OT -> M41T62LC6F; device Microchip_By_element14_Batch_1:MCP73812T-420I/OT -> MyParts:M41T62LC6F
- renumbered C19 to C13, D1 to D2, U$2 to U$13
Connections:
- removed net FTDI_VCC: IC1.VCC, L1.1
- removed net KATHODE: J1.2(LEDCATHODE), R13.1
- removed net N$11: LED5.A, R10.1
- removed net N$20: R10.2, U1.(PCINT23/AIN1)_PD7
- new net INT_RTC: U$1.IQR, U1.(PCINT19/OC2B/INT1)_PD3
- new net N$5: R16.2, U$12.PROG
- new net N$6: R16.1, U$12.VSS
- new net SCL: R5.1, U$1.SCL, U1.PC5_(ADC5/SCL/PCINT13)
- new net SDA: R1.1, U$1.SDA, U1.PC4_(ADC4/SDA/PCINT12)
- net 8: now also IC2.USBDP, R19.1; no longer IC1.USBDP, R7.1
- net 9: now also IC2.USBDM, R18.1; no longer IC1.USBDM, R6.1
- net B0: now also JP1.1; no longer U$3.3, U$3.4
- net B1: now also JP1.2; no longer U$4.3, U$4.4
- net B2: now also JP1.3; no longer U$11.3, U$11.4
- net GND: now also C1.1, C11.2, C12.2, C14.2, C15.2, C16.2, C17.2, IC2.GND, JP4.2, R17.1, U$1.VSS, U$5.3(SPIMODE), U$5.5(GND), X2.4; no longer C1.2, C10.2, C5.1, C6.2, C7.2, C8.2, C9.2, IC1.GND, J1.3(SPIMODE), J1.5(GND), LED5.C, R5.1, X1.4
- net LCD_RESET: now also U$5.7(RST); no longer J1.7(RST)
- net LEDANODE: now also U$5.1(LEDANODE); no longer J1.1(LEDANODE)
- net MOSI: now also U$5.8(SDA); no longer J1.8(SDA)
- net N$1: now also R13.1, U$5.2(LEDCATHODE); no longer R1.2, U$1.PROG
- net N$2: now also IC2.VCC, L2.1; no longer R1.1, U$1.VSS
- net N$26: now also U$5.12; no longer J1.12
- net N$27: now also U$5.11; no longer J1.11
- net NET1: now also C17.1, IC2.!RESET, IC2.3V3OUT, IC2.VCCIO, R20.1, R21.1; no longer C10.1, IC1.!RESET, IC1.3V3OUT, IC1.VCCIO, R8.1, R9.1
- net RXD: now also IC2.TXD, R20.2; no longer IC1.TXD, JP7.1, R8.2
- net SCK: now also U$5.9(SCL); no longer J1.9(SCL)
- net SHEILD: now also X2.5; no longer X1.5
- net SS: now also U$5.6(CS); no longer J1.6(CS)
- net TXD: now also IC2.RXD, R21.2; no longer IC1.RXD, JP6.1, R9.2
- net USB+: now also C2.1, R19.2, X2.3; no longer C6.1, R7.2, X1.3
- net USB-: now also C1.2, R18.2, X2.2; no longer C5.2, R6.2, X1.2
- net VBAT: now also C12.1, U$12.VBAT; no longer C2.1, U$1.VBAT
- net VCC: now also C14.1, C15.1, C16.1, JP4.1, L2.2, R1.2, R5.2, U$1.VCC, U$5.10(D/C), U$5.4(VDD); no longer C7.1, C8.1, C9.1, J1.10(D/C), J1.4(VDD), L1.2, U$11.1, U$11.2, U$3.1, U$3.2, U$4.1, U$4.2
- net VDD: now also R17.2; no longer JP3.4, R5.2
- net VUSB: now also C11.1, U$12.CE, U$12.VDD, X2.1; no longer C1.1, U$1.CE, U$1.VDD, X1.1
Other:
- note added: "Button Inputs"
- note added: "Using external buttons to conserve space on the board"
- note removed: "Charging Circuit With Load Sharing Component"
- note removed: "Extra Serial Connection"
- note removed: "Input Buttons"
- note removed: "USB Connection"
- note removed: "USB to Serial Converter"
- moved on the sheet: C1, C2, R1, R2, R3, R4, R5
